File: KiCad Schematics/dodecahedron_n4.sch (KiCad schematic (older format))
At the start: 65 parts, among them J1 Conn_01x04_Female, U1 IS31FL3733-QF, U2 Board, U3 Board, U4 Jumper4, U5 Jumper4

Commit message: moved files and final order
Parts:
- added R2: 100k, Resistor_SMD:R_0402_1005Metric_Pad0.72x0.64mm_HandSolder, symbol Device:R
- C1, C3: value C -> 470nF
- C2, C4, C5: value C -> 100nF
- R1: value R -> 20k
- R4, R5: value R -> 100k
Connections:
- net VCC: now also R2.1
- net at U1.45 (~INTB): now also R2.2
Changed lines of the file:
@@
 P 7250 -100
 F 0 "C1" V 6998 -100 50  0000 C CNN
-F 1 "C" V 7089 -100 50  0000 C CNN
+F 1 "470nF" V 7089 -100 50  0000 C CNN
 F 2 "Capacitor_SMD:C_0402_1005Metric_Pad0.74x0.62mm_HandSolder" H 7288 -250 50  0001 C CNN
 F 3 "~" H 7250 -100 50  0001 C CNN
@@
 P 6100 -500
 F 0 "R1" H 6170 -454 50  0000 L CNN
-F 1 "R" H 6170 -545 50  0000 L CNN
+F 1 "20k" H 6170 -545 50  0000 L CNN
 F 2 "Resistor_SMD:R_0402_1005Metric_Pad0.72x0.64mm_HandSolder" V 6030 -500 50  0001 C CNN
 F 3 "~" H 6100 -500 50  0001 C CNN
@@
 P 6500 -500
 F 0 "R5" H 6570 -454 50  0000 L CNN
-F 1 "R" H 6570 -545 50  0000 L CNN
+F 1 "100k" H 6570 -545 50  0000 L CNN
 F 2 "Resistor_SMD:R_0402_1005Metric_Pad0.72x0.64mm_HandSolder" V 6430 -500 50  0001 C CNN
 F 3 "~" H 6500 -500 50  0001 C CNN
@@
 P 6400 -500
 F 0 "R4" H 6470 -454 50  0000 L CNN
-F 1 "R" H 6470 -545 50  0000 L CNN
+F 1 "100k" H 6470 -545 50  0000 L CNN
 F 2 "Resistor_SMD:R_0402_1005Metric_Pad0.72x0.64mm_HandSolder" V 6330 -500 50  0001 C CNN
 F 3 "~" H 6400 -500 50  0001 C CNN
@@
 P 7450 600
 F 0 "C2" V 7198 600 50  0000 C CNN
-F 1 "C" V 7289 600 50  0000 C CNN
+F 1 "100nF" V 7289 600 50  0000 C CNN
 F 2 "Capacitor_SMD:C_0402_1005Metric_Pad0.74x0.62mm_HandSolder" H 7488 450 50  0001 C CNN
 F 3 "~" H 7450 600 50  0001 C CNN
@@
 P 7450 700
 F 0 "C3" V 7198 700 50  0000 C CNN
-F 1 "C" V 7289 700 50  0000 C CNN
+F 1 "470nF" V 7289 700 50  0000 C CNN
 F 2 "Capacitor_SMD:C_0402_1005Metric_Pad0.74x0.62mm_HandSolder" H 7488 550 50  0001 C CNN
 F 3 "~" H 7450 700 50  0001 C CNN
@@
 P 7450 800
 F 0 "C4" V 7198 800 50  0000 C CNN
-F 1 "C" V 7289 800 50  0000 C CNN
+F 1 "100nF" V 7289 800 50  0000 C CNN
 F 2 "Capacitor_SMD:C_0402_1005Metric_Pad0.74x0.62mm_HandSolder" H 7488 650 50  0001 C CNN
 F 3 "~" H 7450 800 50  0001 C CNN
@@
 P 7450 900
 F 0 "C5" V 7198 900 50  0000 C CNN
-F 1 "C" V 7289 900 50  0000 C CNN
+F 1 "100nF" V 7289 900 50  0000 C CNN
 F 2 "Capacitor_SMD:C_0402_1005Metric_Pad0.74x0.62mm_HandSolder" H 7488 750 50  0001 C CNN
 F 3 "~" H 7450 900 50  0001 C CNN
@@
 Text GLabel 8500 -2300 2    50   Input ~ 0
 ADDR2
+$Comp
+L Device:R R2
+U 1 1 61BA98A1
+P 6600 -500
+F 0 "R2" H 6670 -454 50  0000 L CNN
+F 1 "100k" H 6670 -545 50  0000 L CNN
+F 2 "Resistor_SMD:R_0402_1005Metric_Pad0.72x0.64mm_HandSolder" V 6530 -500 50  0001 C CNN
+F 3 "~" H 6600 -500 50  0001 C CNN
+	1    6600 -500
+	1    0    0    -1
+$EndComp
+Wire Wire Line
+	6600 -350 6600 0
+$Comp
+L power:VCC #PWR0115
+U 1 1 61BC27E1
+P 6600 -650
+F 0 "#PWR0115" H 6600 -800 50  0001 C CNN
+F 1 "VCC" H 6615 -477 50  0000 C CNN
+F 2 "" H 6600 -650 50  0001 C CNN
+F 3 "" H 6600 -650 50  0001 C CNN
+	1    6600 -650
+	1    0    0    -1
+$EndComp
 $EndSCHEMATC

Commit message: updated PCB
Connections:
- net CS10: now also D25.4 (A)
- net VCC: now also C1.2, U1.39 (VIO)
- net INTB: now reaches R2.2, U1.45 (~INTB)
- net SDB: now reaches R5.2, U1.46 (~SDB)
- net I2C_RST: now reaches R4.2, U1.47 (IICRST)
Other:
- moved on the sheet: D25
Changed lines of the file:
@@
-$EndComp
-$Comp
-L dodecahedron_boards:LED_RBGA D25
-U 1 1 61B4EDA8
-P 5450 4050
-F 0 "D25" H 5450 4547 50  0000 C CNN
-F 1 "LED_RBGA" H 5450 4456 50  0000 C CNN
-F 2 "dodecahedron_n4:B2020RGBA" H 5450 4000 50  0001 C CNN
-F 3 "~" H 5450 4000 50  0001 C CNN
-	1    5450 4050
-	1    0    0    -1
 $EndComp
 $Comp
@@
 	4100 3850 4650 3850
 Connection ~ 4650 3850
-Wire Wire Line
-	4650 3850 5250 3850
-Connection ~ 5250 3850
-Wire Wire Line
-	5250 3850 5750 3850
 Connection ~ 5750 3850
 Wire Wire Line
@@
 	4100 4050 4650 4050
 Connection ~ 4650 4050
-Wire Wire Line
-	4650 4050 5250 4050
-Connection ~ 5250 4050
-Wire Wire Line
-	5250 4050 5750 4050
 Connection ~ 5750 4050
 Wire Wire Line
@@
 Wire Wire Line
 	4650 4250 4100 4250
-Connection ~ 5250 4250
-Wire Wire Line
-	5250 4250 4650 4250
 Connection ~ 5750 4250
-Wire Wire Line
-	5750 4250 5250 4250
 Connection ~ 6300 4250
 Wire Wire Line
@@
 Wire Wire Line
 	6150 4150 6150 3250
-Wire Wire Line
-	5600 5950 5600 3250
 Wire Wire Line
 	5050 5950 5050 4150
@@
 	1    0    0    -1
 $EndComp
+$Comp
+L power:VCC #PWR0116
+U 1 1 61EB73C6
+P 7100 -250
+F 0 "#PWR0116" H 7100 -400 50  0001 C CNN
+F 1 "VCC" H 7115 -77 50  0000 C CNN
+F 2 "" H 7100 -250 50  0001 C CNN
+F 3 "" H 7100 -250 50  0001 C CNN
+	1    7100 -250
+	1    0    0    -1
+$EndComp
+Wire Wire Line
+	7000 -100 7000 -250
+Wire Wire Line
+	7000 -250 7100 -250
+Connection ~ 7000 -100
+Text Label 6500 -100 1    50   ~ 0
+SDB
+Text Label 6400 -50  1    50   ~ 0
+I2C_RST
+Text Label 6600 -100 1    50   ~ 0
+INTB
+$Comp
+L dodecahedron_boards:LED_RBGA D25
+U 1 1 61B4EDA8
+P 5400 4050
+F 0 "D25" H 5400 4547 50  0000 C CNN
+F 1 "LED_RBGA" H 5400 4456 50  0000 C CNN
+F 2 "dodecahedron_n4:B2020RGBA" H 5400 4000 50  0001 C CNN
+F 3 "~" H 5400 4000 50  0001 C CNN
+	1    5400 4050
+	1    0    0    -1
+$EndComp
+Wire Wire Line
+	4650 3850 5200 3850
+Connection ~ 5200 3850
+Wire Wire Line
+	5200 3850 5750 3850
+Connection ~ 5200 4250
+Wire Wire Line
+	5200 4250 4650 4250
+Wire Wire Line
+	5750 4250 5200 4250
+Wire Wire Line
+	4650 4050 5200 4050
+Connection ~ 5200 4050
+Wire Wire Line
+	5200 4050 5750 4050
+Wire Wire Line
+	5600 5950 5600 4150
+Wire Wire Line
+	5600 4150 5600 3250
+Connection ~ 5600 4150
 $EndSCHEMATC

Commit message: kicad and case
Parts:
- added C6: 1uF, Capacitor_SMD:C_0805_2012Metric_Pad1.18x1.45mm_HandSolder, symbol Device:C
- added J2: Conn_01x04_Female, Connector_JST:JST_SH_SM04B-SRSS-TB_1x04-1MP_P1.00mm_Horizontal, symbol Connector:Conn_01x04_Female
Connections:
- net GND: now also C6.1, J2.4 (Pin_4)
- net SCL: now also J2.1 (Pin_1)
- net SDA: now also J2.2 (Pin_2)
- net VCC: now also C6.2, J2.3 (Pin_3)
Changed lines of the file:
@@
 	5600 4150 5600 3250
 Connection ~ 5600 4150
+$Comp
+L Connector:Conn_01x04_Female J2
+U 1 1 6304B0AD
+P 6800 -700
+F 0 "J2" V 6738 -988 50  0000 R CNN
+F 1 "Conn_01x04_Female" V 6647 -988 50  0000 R CNN
+F 2 "Connector_JST:JST_SH_SM04B-SRSS-TB_1x04-1MP_P1.00mm_Horizontal" H 6800 -700 50  0001 C CNN
+F 3 "~" H 6800 -700 50  0001 C CNN
+	1    6800 -700
+	0    -1   -1   0
+$EndComp
+Connection ~ 6700 -500
+Connection ~ 6800 -500
+Connection ~ 6900 -500
+Connection ~ 7000 -500
+$Comp
+L Device:C C6
+U 1 1 630E39E3
+P 8350 -200
+F 0 "C6" V 8098 -200 50  0000 C CNN
+F 1 "1uF" V 8189 -200 50  0000 C CNN
+F 2 "Capacitor_SMD:C_0805_2012Metric_Pad1.18x1.45mm_HandSolder" H 8388 -350 50  0001 C CNN
+F 3 "~" H 8350 -200 50  0001 C CNN
+	1    8350 -200
+	0    1    1    0
+$EndComp
+$Comp
+L power:GND #PWR0117
+U 1 1 630E39ED
+P 8500 -200
+F 0 "#PWR0117" H 8500 -450 50  0001 C CNN
+F 1 "GND" V 8505 -328 50  0000 R CNN
+F 2 "" H 8500 -200 50  0001 C CNN
+F 3 "" H 8500 -200 50  0001 C CNN
+	1    8500 -200
+	0    -1   1    0
+$EndComp
+$Comp
+L power:VCC #PWR0118
+U 1 1 630FBE7B
+P 8200 -200
+F 0 "#PWR0118" H 8200 -350 50  0001 C CNN
+F 1 "VCC" H 8215 -27 50  0000 C CNN
+F 2 "" H 8200 -200 50  0001 C CNN
+F 3 "" H 8200 -200 50  0001 C CNN
+	1    8200 -200
+	1    0    0    -1
+$EndComp
 $EndSCHEMATC
