File: KiCad Schematics/dodecahedron_n4.kicad_pcb (KiCad board)
At the start: 4 copper layers, 32.5 x 30.9 mm, 67 parts, among them J1 Conn_01x04_Female, U1 IS31FL3733-QF, U2 Board, U3 Board, U4 Jumper4, U5 Jumper4

Commit message: moved files and final order
Parts:
- added R2: 100k, Resistor_SMD:R_0402_1005Metric_Pad0.72x0.64mm_HandSolder, B.Cu at (90.6, 55.9)
- C1, C3: value C -> 470nF
- C2, C4, C5: value C -> 100nF
- R1: value R -> 20k
- R4, R5: value R -> 100k
- moved R5 0.55 mm to (89.6, 55.9)
- moved R4 0.51 mm to (88.6, 55.9)
- moved U5 0.13 mm to (92.0, 54.9)
- moved U4 0.06 mm to (94.2, 55.0)
Routing:
- net Net-(R2-Pad2): track 0.00 -> 5.38 mm
- net VCC: track 31.5 -> 33.7 mm, vias 10 -> 11
- net GND: track 40.1 -> 39.6 mm, vias 27 -> 28

Commit message: updated PCB
Parts:
- removed kibuzzard-61B81406, kibuzzard-61B81B90: G***, label
Connections:
- net Net-(R2-Pad2) renamed /INTB
- net Net-(R4-Pad2) renamed /I2C_RST
- net Net-(R5-Pad2) renamed /SDB
- C1 pad 2: Net-(C1-Pad2) -> VCC
- D25 pad 4: Net-(D25-Pad4) -> /CS10
- U1 pad 39: Net-(C1-Pad2) -> VCC
Routing:
- net /CS10: track 31.3 -> 35.2 mm
- net VCC: track 33.7 -> 35.7 mm
- net Net-(C1-Pad2): track 1.62 -> 0.00 mm

Commit message: kicad and case
Parts:
- added C6: 1uF, Capacitor_SMD:C_0805_2012Metric_Pad1.18x1.45mm_HandSolder, B.Cu at (76.8, 43.2)
- added J2: Conn_01x04_Female, Connector_JST:JST_SH_SM04B-SRSS-TB_1x04-1MP_P1.00mm_Horizontal, B.Cu at (73.9, 49.4)
- moved C5 6.80 mm to (73.3, 44.5)
Routing:
- net SDA: track 23.8 -> 47.7 mm, vias 2 -> 3
- net SCL: track 26.3 -> 46.9 mm, vias 0 -> 2
- net VCC: track 35.7 -> 46.2 mm, vias 11 -> 12
- net GND: track 39.6 -> 47.8 mm
- net /CS5: track 27.3 -> 25.7 mm, vias 4 -> 5
- net /CS8: track 35.0 -> 33.6 mm
- net /CS3: track 35.1 -> 35.7 mm

Commit message: reworking lost progress
Other:
- net class Default removed
